File: examples/audio_player_project/main.kicad_pcb (KiCad board)
At the start: 6 copper layers, 75 x 45 mm, 0 parts

Commit message: Fix native KiCad audio validation path
Other:
- board text added: "Analog_Region"
- board text added: "Digital_Region"
Changed lines of the file:
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@@
     (add_net "SPK_R-")
   )
-  (zone (net 0) (net_name "") (layers "Cmts.User")
-    (name "Digital_Region")
-    (hatch edge 0.5)
-    (connect_pads yes)
-    (min_thickness 0.15)
-    (fill no (thermal_gap 0.5) (thermal_bridge_width 0.5))
-    (polygon
-      (pts
-        (xy 0.0 22.5) (xy 75.0 22.5) (xy 75.0 45.0) (xy 0.0 45.0)
-      )
-    )
+  (gr_rect
+    (start 0.0 22.5)
+    (end 75.0 45.0)
+    (stroke (width 0.15) (type dash))
+    (fill none)
+    (layer "Cmts.User")
   )
-  (zone (net 0) (net_name "") (layers "Cmts.User")
-    (name "Analog_Region")
-    (hatch edge 0.5)
-    (connect_pads yes)
-    (min_thickness 0.15)
-    (fill no (thermal_gap 0.5) (thermal_bridge_width 0.5))
-    (polygon
-      (pts
-        (xy 0.0 0.0) (xy 75.0 0.0) (xy 75.0 22.5) (xy 0.0 22.5)
-      )
-    )
+  (gr_text "Digital_Region"
+    (at 1.0 44.0 0)
+    (layer "Cmts.User")
+    (effects (font (size 1.5 1.5)) (justify left bottom))
+  )
+  (gr_rect
+    (start 0.0 0.0)
+    (end 75.0 22.5)
+    (stroke (width 0.15) (type dash))
+    (fill none)
+    (layer "Cmts.User")
+  )
+  (gr_text "Analog_Region"
+    (at 1.0 21.5 0)
+    (layer "Cmts.User")
+    (effects (font (size 1.5 1.5)) (justify left bottom))
   )
   (zone (net 0) (net_name "") (layers "F.Cu")
